Commit message: Added Gazebo simulation. Physics OK!

File: install/robot/share/robot/urdf/big_arm.urdf (robot description, URDF)
Before this commit: robot big_arm, 15 links, 14 joints
Joints:
- joint joint_12: limit lower=0 upper=6.183 effort=1000 velocity=10 -> lower=0 upper=6.31 effort=1000 velocity=10
- joint joint_6_g1: limit lower=0 upper=6.183 effort=1000 velocity=10 -> lower=0 upper=0 effort=1000 velocity=10
- joint joint_6_g2: limit lower=0 upper=6.183 effort=1000 velocity=10 -> lower=0 upper=0 effort=1000 velocity=10
- joint joint_6_g3: limit lower=0 upper=6.183 effort=1000 velocity=10 -> lower=0 upper=0 effort=1000 velocity=10
- joint joint_6_g4: limit lower=0 upper=6.183 effort=1000 velocity=10 -> lower=0 upper=0 effort=1000 velocity=10
- joint joint_base_1: limit lower=0 upper=6.183 effort=1000 velocity=10 -> lower=-3.14159 upper=3.14159 effort=1000 velocity=10
- joint joint_grip_1b: limit lower=0 upper=6.183 effort=1000 velocity=10 -> lower=0 upper=0 effort=1000 velocity=10
- joint joint_grip_2b: limit lower=0 upper=6.183 effort=1000 velocity=10 -> lower=0 upper=0 effort=1000 velocity=10
- joint joint_grip_3b: limit lower=0 upper=6.183 effort=1000 velocity=10 -> lower=0 upper=0 effort=1000 velocity=10
- joint joint_grip_4b: limit lower=0 upper=6.183 effort=1000 velocity=10 -> lower=0 upper=0 effort=1000 velocity=10

Commit message: Implementing effort controller for each joint

File: install/robot/share/robot/urdf/big_arm.urdf (robot description, URDF)
Before this commit: robot big_arm, 15 links, 14 joints
Links:
- added link world
- link base_link: mass 25.4419917555561 -> 2.4419917555561
Joints:
- added joint world_joint: type fixed, parent world, child base_link, origin xyz=0.0 0.0 0.0 rpy=0.0 0.0 0.0
- joint joint_12: limit lower=0 upper=6.31 effort=1000 velocity=10 -> lower=0 upper=0 effort=10000 velocity=10
- joint joint_23: limit lower=0 upper=6.183 effort=1000 velocity=10 -> lower=0 upper=0 effort=1000 velocity=10
- joint joint_34: limit lower=0 upper=6.183 effort=1000 velocity=10 -> lower=0 upper=0 effort=1000 velocity=10
- joint joint_45: limit lower=0 upper=6.183 effort=1000 velocity=10 -> lower=0 upper=0 effort=1000 velocity=10
- joint joint_56: limit lower=0 upper=6.183 effort=1000 velocity=10 -> lower=0 upper=0 effort=1000 velocity=10
- joint joint_base_1: limit lower=-3.14159 upper=3.14159 effort=1000 velocity=10 -> lower=-3.14159 upper=3.14159 effort=10000 velocity=10

Commit message: First joint basic controller

File: install/robot/share/robot/urdf/big_arm.urdf (robot description, URDF)
Before this commit: robot big_arm, 16 links, 15 joints
Joints:
- joint joint_base_1: limit lower=-3.14159 upper=3.14159 effort=10000 velocity=10 -> lower=-3.14159 upper=3.14159 effort=100 velocity=10

Commit message: Developing a new model

File: install/robot/share/robot/urdf/big_arm.urdf (robot description, URDF)
Before this commit: robot big_arm, 16 links, 15 joints
Links:
- link link_1: mass 1.24036308689963 -> 2.24036308689963
Joints:
- joint joint_12: limit lower=0 upper=0 effort=10000 velocity=10 -> lower=-3.14159 upper=3.14159 effort=10000 velocity=10; origin xyz=0 0 0.11 rpy=-1.5708 -0.95024 -3.0507 -> xyz=0 0 0.11 rpy=-1.5708 0 -3.14159
- joint joint_23: limit lower=0 upper=0 effort=1000 velocity=10 -> lower=-3.14159 upper=3.14159 effort=1000 velocity=10; origin xyz=0.38 0 0 rpy=0 0 -1.207 -> xyz=0.38 0 0 rpy=0 0 -1.57079
- joint joint_34: limit lower=0 upper=0 effort=1000 velocity=10 -> lower=0 upper=6.183 effort=1000 velocity=10; origin xyz=0.38 0 0 rpy=0 -0.090932 -0.98436 -> xyz=0.38 0 0 rpy=0 0 -1.57079
- joint joint_45: limit lower=0 upper=0 effort=1000 velocity=10 -> lower=0 upper=6.183 effort=1000 velocity=10; origin xyz=0.37701 -0.032936 -0.034377 rpy=0.062559 -0.066036 2.3822 -> xyz=0.37701 0 0 rpy=0 0 3.14159
- joint joint_56: limit lower=0 upper=0 effort=1000 velocity=10 -> lower=0 upper=6.183 effort=1000 velocity=10
- joint joint_base_1: limit lower=-3.14159 upper=3.14159 effort=100 velocity=10 -> lower=-3.14159 upper=3.14159 effort=10000 velocity=10

File: install/robot/share/robot/urdf/big_arm_servos.urdf (robot description, URDF)
Before this commit: robot big_arm_servos, 16 links, 15 joints
Joints:
- joint joint_23: origin xyz=0.38 0 0 rpy=0 0 -1.5 -> xyz=0.38 0 0 rpy=0 0 -1.57079
- joint joint_45: origin xyz=0.37701 -0.032936 0 rpy=0 -0.066036 3.14159 -> xyz=0.37701 0 0 rpy=0 0 3.14159

File: src/robot/urdf/big_arm_servos.urdf (robot description, URDF)
Before this commit: robot big_arm_servos, 16 links, 15 joints
Joints:
- joint joint_23: origin xyz=0.38 0 0 rpy=0 0 -1.5 -> xyz=0.38 0 0 rpy=0 0 -1.57079
- joint joint_45: origin xyz=0.37701 -0.032936 -0.034377 rpy=0 -0.066036 3.14159 -> xyz=0.37701 0 0 rpy=0 0 3.14159
