Commit message: Multipoint action server for trajectories

File: install/robot/share/robot/urdf/big_arm_servos.urdf (robot description, URDF)
Before this commit: robot big_arm_servos, 4 links, 3 joints
Links:
- added link grip_1, mass 0.11992363568227; collision mesh filename=package://robot/meshes/grip_1.STL; visual mesh filename=package://robot/meshes/grip_1.STL
- added link grip_1b, mass 0.141643537240913; collision mesh filename=package://robot/meshes/grip_1b.STL; visual mesh filename=package://robot/meshes/grip_1b.STL
- added link grip_2, mass 0.119923642785374; collision mesh filename=package://robot/meshes/grip_2.STL; visual mesh filename=package://robot/meshes/grip_2.STL
- added link grip_2b, mass 0.141643614685743; collision mesh filename=package://robot/meshes/grip_2b.STL; visual mesh filename=package://robot/meshes/grip_2b.STL
- added link grip_3, mass 0.119923637058051; collision mesh filename=package://robot/meshes/grip_3.STL; visual mesh filename=package://robot/meshes/grip_3.STL
- added link grip_3b, mass 0.141643615845273; collision mesh filename=package://robot/meshes/grip_3b.STL; visual mesh filename=package://robot/meshes/grip_3b.STL
- added link grip_4, mass 0.119923640551901; collision mesh filename=package://robot/meshes/grip_4.STL; visual mesh filename=package://robot/meshes/grip_4.STL
- added link grip_4b, mass 0.141643613852148; collision mesh filename=package://robot/meshes/grip_4b.STL; visual mesh filename=package://robot/meshes/grip_4b.STL
- added link link_3, mass 0.492773406896242; collision mesh filename=package://robot/meshes/link_3.STL; visual mesh filename=package://robot/meshes/link_3.STL
- added link link_4, mass 1.38058358126134; collision mesh filename=package://robot/meshes/link_4.STL; visual mesh filename=package://robot/meshes/link_4.STL
- added link link_5, mass 0.130378439395373; collision mesh filename=package://robot/meshes/link_5.STL; visual mesh filename=package://robot/meshes/link_5.STL
- added link link_6, mass 0.665759903912911; collision mesh filename=package://robot/meshes/link_6.STL; visual mesh filename=package://robot/meshes/link_6.STL
Joints:
- added joint joint_23: type revolute, parent link_2, child link_3, origin xyz=0.38 0 0 rpy=0 0 -1.207, axis 0 0 1, limit lower=0 upper=6.183 effort=1000 velocity=10
- added joint joint_34: type revolute, parent link_3, child link_4, origin xyz=0.38 0 0 rpy=0 -0.090932 -0.98436, axis 0 0 1, limit lower=0 upper=6.183 effort=1000 velocity=10
- added joint joint_45: type revolute, parent link_4, child link_5, origin xyz=0.37701 -0.032936 -0.034377 rpy=0.062559 -0.066036 2.3822, axis 0 0 1, limit lower=0 upper=6.183 effort=1000 velocity=10
- added joint joint_56: type revolute, parent link_5, child link_6, origin xyz=-0.04 0 0.002 rpy=-2.3654 1.5708 0.77614, axis 0 0 1, limit lower=0 upper=6.183 effort=1000 velocity=10
- added joint joint_6_g1: type revolute, parent link_6, child grip_1, origin xyz=-0.011072 0.05897 0.091 rpy=-1.7211 -0.33932 1.7564, axis 0 0 1, limit lower=0 upper=0 effort=1000 velocity=10
- added joint joint_6_g2: type revolute, parent link_6, child grip_2, origin xyz=0.05897 0.011072 0.091 rpy=-1.5708 -0.19278 0.1856, axis 0 0 1, limit lower=0 upper=0 effort=1000 velocity=10
- added joint joint_6_g3: type revolute, parent link_6, child grip_3, origin xyz=0.011072 -0.05897 0.091 rpy=-1.5491 -0.33932 -1.3852, axis 0 0 1, limit lower=0 upper=0 effort=1000 velocity=10
- added joint joint_6_g4: type revolute, parent link_6, child grip_4, origin xyz=-0.05897 -0.011072 0.091 rpy=1.5708 -0.4026 -2.956, axis 0 0 1, limit lower=0 upper=0 effort=1000 velocity=10
- added joint joint_grip_1b: type revolute, parent grip_1, child grip_1b, origin xyz=0.11 0 0 rpy=0.011605 0.14985 -1.4932, axis 0 0 1, limit lower=0 upper=0 effort=1000 velocity=10
- added joint joint_grip_2b: type revolute, parent grip_2, child grip_2b, origin xyz=0.10759 -0.022911 0 rpy=0 0 -1.5817, axis 0 0 1, limit lower=0 upper=0 effort=1000 velocity=10
- added joint joint_grip_3b: type revolute, parent grip_3, child grip_3b, origin xyz=0.11 0 0 rpy=-0.013124 -0.017244 -0.9202, axis 0 0 1, limit lower=0 upper=0 effort=1000 velocity=10
- added joint joint_grip_4b: type revolute, parent grip_4, child grip_4b, origin xyz=0.11 0 0 rpy=3.1416 0 1.2805, axis 0 0 1, limit lower=0 upper=0 effort=1000 velocity=10

Commit message: Stable commit

File: install/robot/share/robot/urdf/big_arm_servos.urdf (robot description, URDF)
Before this commit: robot big_arm_servos, 16 links, 15 joints
Joints:
- joint joint_12: origin xyz=0 0 0.11 rpy=-1.5708 -0.95024 -3.0507 -> xyz=0 0 0.11 rpy=-1.5708 0 -3.0507
- joint joint_23: limit lower=0 upper=6.183 effort=1000 velocity=10 -> lower=-3.14159 upper=3.14159 effort=1000 velocity=10; origin xyz=0.38 0 0 rpy=0 0 -1.207 -> xyz=0.38 0 0 rpy=0 0 -1.57079
- joint joint_34: origin xyz=0.38 0 0 rpy=0 -0.090932 -0.98436 -> xyz=0.38 0 0 rpy=0 -0.090932 -1.57079
- joint joint_45: origin xyz=0.37701 -0.032936 -0.034377 rpy=0.062559 -0.066036 2.3822 -> xyz=0.37701 -0.032936 -0.034377 rpy=0 0 3.14159

Commit message: Fixing transforms

File: install/robot/share/robot/urdf/big_arm_servos.urdf (robot description, URDF)
Before this commit: robot big_arm_servos, 16 links, 15 joints
Joints:
- joint joint_12: origin xyz=0 0 0.11 rpy=-1.5708 0 -3.0507 -> xyz=0 0 0.11 rpy=-1.5708 0 -3.14159
- joint joint_23: origin xyz=0.38 0 0 rpy=0 0 -1.57079 -> xyz=0.38 0 0 rpy=0 0 -1.5
- joint joint_34: origin xyz=0.38 0 0 rpy=0 -0.090932 -1.57079 -> xyz=0.38 0 0 rpy=0 0 -1.57079
- joint joint_45: origin xyz=0.37701 -0.032936 -0.034377 rpy=0 0 3.14159 -> xyz=0.37701 -0.032936 0 rpy=0 -0.066036 3.14159

File: src/robot/urdf/big_arm_servos.urdf (robot description, URDF)
Before this commit: robot big_arm_servos, 16 links, 15 joints
Joints:
- joint joint_12: origin xyz=0 0 0.11 rpy=-1.5708 0 -3.0507 -> xyz=0 0 0.11 rpy=-1.5708 0 -3.14159
- joint joint_23: origin xyz=0.38 0 0 rpy=0 0 -1.57079 -> xyz=0.38 0 0 rpy=0 0 -1.5
- joint joint_34: origin xyz=0.38 0 0 rpy=0 -0.090932 -1.57079 -> xyz=0.38 0 0 rpy=0 0 -1.57079
- joint joint_45: origin xyz=0.37701 -0.032936 -0.034377 rpy=0 0 3.14159 -> xyz=0.37701 -0.032936 -0.034377 rpy=0 -0.066036 3.14159

Commit message: Added camera sensor for the robot

File: install/robot/share/robot/urdf/big_arm_servos.urdf (robot description, URDF)
Before this commit: robot big_arm_servos, 16 links, 15 joints
Links:
- added link camera_link, mass 0.03; collision box size=0.02 0.02 0.02; visual box size=0.02 0.02 0.02
Joints:
- added joint camera_joint: type fixed, parent link_1, child camera_link, origin xyz=0.15 0.0 0.05 rpy=0.0 0.0 0.0
