Commit message: Fixed URDF and Inverse Kinematics without constraints working fine.

File: src/robot/urdf/big_arm_servos.urdf (robot description, URDF)
Before this commit: robot big_arm_servos, 17 links, 16 joints
Joints:
- joint joint_56: origin xyz=-0.04 0 0.002 rpy=-2.3654 1.5708 -0.7853981634 -> xyz=0 0 0.002 rpy=-2.3654 1.5708 -0.7853981634

Commit message: Added camera and IK works properly. (Merge with main)

File: src/robot/urdf/big_arm_servos.urdf (robot description, URDF)
Before this commit: robot big_arm_servos, 17 links, 16 joints
Links:
- removed link grip_1
- removed link grip_1b
- removed link grip_3
- removed link grip_3b
Joints:
- removed joint joint_6_g1
- removed joint joint_6_g3
- removed joint joint_grip_1b
- removed joint joint_grip_3b
- joint camera_joint: origin xyz=0.15 0.0 0.05 rpy=0.0 0.0 0.0 -> xyz=-0.155 0.0 0.05 rpy=0.0 0.0 3.14159
- joint joint_45: origin xyz=0.37701 0 0 rpy=0 0 3.14159 -> xyz=0.37701 0 0 rpy=0 0 -1.57079
- joint joint_6_g2: limit lower=0 upper=0 effort=1000 velocity=10 -> lower=-3.14159 upper=3.14159 effort=1000 velocity=10
- joint joint_6_g4: limit lower=0 upper=0 effort=1000 velocity=10 -> lower=-3.14159 upper=3.14159 effort=1000 velocity=10
- joint joint_grip_2b: limit lower=0 upper=0 effort=1000 velocity=10 -> lower=-3.14159 upper=3.14159 effort=1000 velocity=10
- joint joint_grip_4b: limit lower=0 upper=0 effort=1000 velocity=10 -> lower=-3.14159 upper=3.14159 effort=1000 velocity=10

Commit message: Merged fix_urdf with main

File: src/robot/urdf/big_arm_servos.urdf (robot description, URDF)
Before this commit: robot big_arm_servos, 13 links, 12 joints
Joints:
- joint camera_joint: origin xyz=0.15 0.0 0.05 rpy=0.0 0.0 0.0 -> xyz=-0.155 0.0 0.05 rpy=0.0 0.0 3.14159
